Commit message: Update fishbot URDF description Mass/Inertia

File: chapt6_ws/src/fishbot_description/urdf/fishbot/actuator/caster.urdf.xacro (robot description, xacro)
@@ -1,4 +1,5 @@
 <?xml version="1.0"?>
 <robot xmlns:xacro="http://www.ros.org/wiki/xacro" name='first_robot'>
+    <xacro:include filename="$(find fishbot_description)/urdf/fishbot/common_inertia.xacro"/>
     <xacro:macro name="caster_xacro" params="caster_name xyz">
         <link name='${caster_name}_link'>
@@ -16,5 +17,18 @@
                 </material>
             </visual>
+            <xacro:box_inertia m="0.1" w="0.02" h="0.10" d="0.02"/>
         </link>
+        <collision>
+            <!-- 沿自己几何中心的坐标系 -->
+            <origin xyz="0.0 0.0 0.0" rpy="0.0 0.0 0.0"/>
+            <!-- 几何形状 -->
+            <geometry>
+                <sphere radius="0.016"/>
+            </geometry>
+            <!-- 颜色  -->
+            <material name="yellow">
+                <color rgba="1.0 1.0 0.0 0.8"/>
+            </material>
+        </collision>
         <!-- 机器人关节 用于组合机器人的部件-->
         <joint name='${caster_name}_joint' type='fixed'>
@@ -23,4 +37,5 @@
             <origin xyz="${xyz}" rpy="0.0 0.0 0.0"/>
         </joint>
+        <xacro:sphere_inertia m="0.05" r="0.016"/>
     </xacro:macro>
 </robot>

File: chapt6_ws/src/fishbot_description/urdf/fishbot/actuator/wheel.urdf.xacro (robot description, xacro)
@@ -1,4 +1,5 @@
 <?xml version="1.0"?>
 <robot xmlns:xacro="http://www.ros.org/wiki/xacro" name='first_robot'>
+    <xacro:include filename="$(find fishbot_description)/urdf/fishbot/common_inertia.xacro"/>
     <xacro:macro name="wheel_xacro" params="wheel_name xyz">
         <link name='${wheel_name}_link'>
@@ -16,4 +17,17 @@
                 </material>
             </visual>
+            <collision>
+                <!-- 沿自己几何中心的坐标系 -->
+                <origin xyz="0.0 0.0 0.0" rpy="1.57079 0.0 0.0"/>
+                <!-- 几何形状 -->
+                <geometry>
+                    <cylinder radius="0.032" length="0.04"/>
+                </geometry>
+                <!-- 颜色  -->
+                <material name="yellow">
+                    <color rgba="1.0 1.0 0.0 0.8"/>
+                </material>
+            </collision>
+            <xacro:cylinder_inertia m="0.05" r="0.032" h="0.04"/>
         </link>
         <!-- 机器人关节 用于组合机器人的部件-->

File: chapt6_ws/src/fishbot_description/urdf/fishbot/base.urdf.xacro (robot description, xacro)
@@ -1,4 +1,5 @@
 <?xml version="1.0"?>
 <robot xmlns:xacro="http://www.ros.org/wiki/xacro" name='first_robot'>
+    <xacro:include filename="$(find fishbot_description)/urdf/fishbot/common_inertia.xacro"/>
     <xacro:macro name="base_xacro" params="length radius">
         <link name="base_footprint"/>
@@ -18,4 +19,17 @@
                 </material>
             </visual>
+            <collision>
+                <!-- 沿自己几何中心的坐标系 -->
+                <origin xyz="0.0 0.0 0.0" rpy="0.0 0.0 0.0"/>
+                <!-- 几何形状 -->
+                <geometry>
+                    <cylinder radius="${radius}" length="${length}"/>
+                </geometry>
+                <!-- 颜色  -->
+                <material name="white">
+                    <color rgba="1.0 1.0 1.0 0.5"/>
+                </material>
+            </collision>
+            <xacro:cylinder_inertia m="1.0" r="${radius}" h="${length}"/>
         </link>
         <joint name='joint_name' type='fixed'>

File: chapt6_ws/src/fishbot_description/urdf/fishbot/sensor/camera.urdf.xacro (robot description, xacro)
@@ -1,4 +1,5 @@
 <?xml version="1.0"?>
 <robot xmlns:xacro="http://www.ros.org/wiki/xacro" name='first_robot'>
+    <xacro:include filename="$(find fishbot_description)/urdf/fishbot/common_inertia.xacro"/>
     <xacro:macro name="camera_xacro" params="xyz">
         <link name='camera_link'>
@@ -16,4 +17,17 @@
                 </material>
             </visual>
+            <collision>
+                <!-- 沿自己几何中心的坐标系 -->
+                <origin xyz="0.0 0.0 0.0" rpy="0.0 0.0 0.0"/>
+                <!-- 几何形状 -->
+                <geometry>
+                    <box size="0.02 0.10 0.02"/>
+                </geometry>
+                <!-- 颜色  -->
+                <material name="black">
+                    <color rgba="0.0 0.0 0.0 0.5"/>
+                </material>
+            </collision>
+            <xacro:box_inertia m="0.05" w="0.02" h="0.02" d="0.02"/>
         </link>
         <!-- 机器人关节 用于组合机器人的部件-->

File: chapt6_ws/src/fishbot_description/urdf/fishbot/sensor/imu.urdf.xacro (robot description, xacro)
@@ -1,4 +1,5 @@
 <?xml version="1.0"?>
 <robot xmlns:xacro="http://www.ros.org/wiki/xacro" name='first_robot'>
+    <xacro:include filename="$(find fishbot_description)/urdf/fishbot/common_inertia.xacro"/>
     <xacro:macro name="imu_xacro" params="xyz">
         <link name='imu_link'>
@@ -16,4 +17,17 @@
                 </material>
             </visual>
+            <collision>
+                <!-- 沿自己几何中心的坐标系 -->
+                <origin xyz="0.0 0.0 0.0" rpy="0.0 0.0 0.0"/>
+                <!-- 几何形状 -->
+                <geometry>
+                    <box size="0.02 0.02 0.02"/>
+                </geometry>
+                <!-- 颜色  -->
+                <material name="black">
+                    <color rgba="0.0 0.0 0.0 0.5"/>
+                </material>
+            </collision>
+            <xacro:box_inertia m="0.05" w="0.02" h="0.02" d="0.02"/>
         </link>
         <!-- 机器人关节 用于组合机器人的部件-->

File: chapt6_ws/src/fishbot_description/urdf/fishbot/sensor/laser.urdf.xacro (robot description, xacro)
@@ -1,4 +1,5 @@
 <?xml version="1.0"?>
 <robot xmlns:xacro="http://www.ros.org/wiki/xacro" name='first_robot'>
+    <xacro:include filename="$(find fishbot_description)/urdf/fishbot/common_inertia.xacro"/>
     <xacro:macro name="laser_xacro" params="xyz">
         <!-- 雷达支撑杆 -->
@@ -17,4 +18,17 @@
                 </material>
             </visual>
+            <collision>
+                <!-- 沿自己几何中心的坐标系 -->
+                <origin xyz="0.0 0.0 0.0" rpy="0.0 0.0 0.0"/>
+                <!-- 几何形状 -->
+                <geometry>
+                    <cylinder radius="0.01" length="0.10"/>
+                </geometry>
+                <!-- 颜色  -->
+                <material name="black">
+                    <color rgba="0.0 0.0 0.0 1.0"/>
+                </material>
+            </collision>
+            <xacro:cylinder_inertia m="0.05" r="0.01" h="0.10"/>
         </link>
         <!-- 雷达 -->
@@ -33,4 +47,17 @@
                 </material>
             </visual>
+            <collision>
+                <!-- 沿自己几何中心的坐标系 -->
+                <origin xyz="0.0 0.0 0.0" rpy="0.0 0.0 0.0"/>
+                <!-- 几何形状 -->
+                <geometry>
+                    <cylinder radius="0.02" length="0.02"/>
+                </geometry>
+                <!-- 颜色  -->
+                <material name="black">
+                    <color rgba="0.0 0.0 0.0 1.0"/>
+                </material>
+            </collision>
+            <xacro:cylinder_inertia m="0.10" r="0.02" h="0.02"/>
         </link>
         <!-- 机器人关节 用于组合机器人的部件-->

Commit message: Gazebo&URDF

File: chapt6_ws/src/fishbot_description/urdf/fishbot/actuator/caster.urdf.xacro (robot description, xacro)
@@ -17,18 +17,24 @@
                 </material>
             </visual>
+            <collision>
+                <!-- 沿自己几何中心的坐标系 -->
+                <origin xyz="0.0 0.0 0.0" rpy="0.0 0.0 0.0"/>
+                <!-- 几何形状 -->
+                <geometry>
+                    <sphere radius="0.016"/>
+                </geometry>
+                <!-- 颜色  -->
+                <material name="yellow">
+                    <color rgba="1.0 1.0 0.0 0.8"/>
+                </material>
+            </collision>
             <xacro:box_inertia m="0.1" w="0.02" h="0.10" d="0.02"/>
         </link>
-        <collision>
-            <!-- 沿自己几何中心的坐标系 -->
-            <origin xyz="0.0 0.0 0.0" rpy="0.0 0.0 0.0"/>
-            <!-- 几何形状 -->
-            <geometry>
-                <sphere radius="0.016"/>
-            </geometry>
-            <!-- 颜色  -->
-            <material name="yellow">
-                <color rgba="1.0 1.0 0.0 0.8"/>
-            </material>
-        </collision>
+        <gazebo reference="${caster_name}_caster_link">
+            <mu1 value="0.0" />
+            <mu2 value="0.0" />
+            <kp value="1000000000.0" />
+            <kd value="1.0" />
+        </gazebo>
         <!-- 机器人关节 用于组合机器人的部件-->
         <joint name='${caster_name}_joint' type='fixed'>
@@ -37,5 +43,4 @@
             <origin xyz="${xyz}" rpy="0.0 0.0 0.0"/>
         </joint>
-        <xacro:sphere_inertia m="0.05" r="0.016"/>
     </xacro:macro>
 </robot>

File: chapt6_ws/src/fishbot_description/urdf/fishbot/actuator/wheel.urdf.xacro (robot description, xacro)
@@ -38,4 +38,10 @@
             <axis xyz="0 1 0"/>
         </joint>
+        <gazebo reference="${wheel_name}_wheel_link">
+            <mu1 value="20.0" />
+            <mu2 value="20.0" />
+            <kp value="1000000000.0" />
+            <kd value="1.0" />
+        </gazebo>
     </xacro:macro>
 </robot>

File: chapt6_ws/src/fishbot_description/urdf/fishbot/sensor/laser.urdf.xacro (robot description, xacro)
@@ -74,4 +74,10 @@
             <origin xyz="${xyz}" rpy="0.0 0.0 0.0"/>
         </joint>
+        <gazebo reference="laser_cylinder_link">
+            <material>Gazebo/Black</material>
+        </gazebo>
+        <gazebo reference="laser_link">
+            <material>Gazebo/Black</material>
+        </gazebo>
     </xacro:macro>
 </robot>
