Commit message: add camera_optical

File: chapt6_ws/src/fishbot_description/urdf/fishbot/plugins/gazebo_sensor_plugin.xacro (robot description, xacro)
@@ -16,5 +16,5 @@
                 <update_rate>5</update_rate>
                 <pose>0 0 0 0 0 0</pose>
-				 <!-- 激光传感器配置 -->
+								<!-- 激光传感器配置 -->
                 <ray>
                     <!-- 设置扫描范围 -->

File: chapt6_ws/src/fishbot_description/urdf/fishbot/sensor/camera.urdf.xacro (robot description, xacro)
@@ -1,39 +1,38 @@
 <?xml version="1.0"?>
-<robot xmlns:xacro="http://www.ros.org/wiki/xacro" name='first_robot'>
-    <xacro:include filename="$(find fishbot_description)/urdf/fishbot/common_inertia.xacro"/>
+<robot xmlns:xacro="http://www.ros.org/wiki/xacro">
+   <xacro:include filename="$(find fishbot_description)/urdf/fishbot/common_inertia.xacro" />
     <xacro:macro name="camera_xacro" params="xyz">
-        <link name='camera_link'>
-            <!-- 部件的外观描述 -->
+        <!-- ============相机模块================ -->
+        <link name="camera_link">
             <visual>
-                <!-- 沿自己几何中心的坐标系 -->
-                <origin xyz="0.0 0.0 0.0" rpy="0.0 0.0 0.0"/>
-                <!-- 几何形状 -->
+                <origin xyz="0 0 0.0" rpy="0 0 0" />
                 <geometry>
-                    <box size="0.02 0.10 0.02"/>
+                    <box size="0.02 0.10 0.02" />
                 </geometry>
-                <!-- 颜色  -->
                 <material name="black">
-                    <color rgba="0.0 0.0 0.0 0.5"/>
+                    <color rgba="0.0 0.0 0.0 0.8"/>
                 </material>
             </visual>
             <collision>
-                <!-- 沿自己几何中心的坐标系 -->
-                <origin xyz="0.0 0.0 0.0" rpy="0.0 0.0 0.0"/>
-                <!-- 几何形状 -->
+                <origin xyz="0 0 0.0" rpy="0 0 0" />
                 <geometry>
-                    <box size="0.02 0.10 0.02"/>
+                    <box size="0.02 0.10 0.02" />
                 </geometry>
-                <!-- 颜色  -->
                 <material name="black">
-                    <color rgba="0.0 0.0 0.0 0.5"/>
+                    <color rgba="0.0 0.0 0.0 0.8"/>
                 </material>
             </collision>
-            <xacro:box_inertia m="0.05" w="0.02" h="0.02" d="0.02"/>
+            <xacro:box_inertia m="0.01" w="0.02" h="0.10" d="0.02" />
         </link>
-        <!-- 机器人关节 用于组合机器人的部件-->
-        <joint name='camera_joint' type='fixed'>
-            <parent link='base_link'/>
-            <child link='camera_link'/>
-            <origin xyz="${xyz}" rpy="0.0 0.0 0.0"/>
+        <link name="camera_optical_link"></link>
+        <joint name="camera_optical_joint" type="fixed">
+            <parent link="camera_link" />
+            <child link="camera_optical_link" />
+            <origin xyz="0 0 0" rpy="${-pi/2} 0 ${-pi/2}" />
+        </joint>
+        <joint name="camera_joint" type="fixed">
+            <parent link="base_link" />
+            <child link="camera_link" />
+            <origin xyz="${xyz}" />
         </joint>
     </xacro:macro>
